File: Jupiter-II.sch (KiCad schematic (older format))
At the start: 49 parts, among them J1 EXPANSION, J2 KEYBOARD, J3 TAPE, J5 9Vdc, SW1 SW_Push, U1 6116, U2 27C64, U3 Z80CPU, U4 74LS367, U5 GAL22V10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

Commit message: Inverted video option
Parts:
- added D11: 5V1, Diodes_THT:D_DO-35_SOD27_P2.54mm_Vertical_KathodeUp, symbol Device:D_Zener_ALT
- added R56: 330, Resistors_SMD:R_0805_HandSoldering, symbol Device:R
Connections:
- net EAR: now also D11.1 (K), R56.2; no longer C7.2
- net GNDD: now also D11.2 (A)
- new net: C7.2, R56.1
Other:
- note removed: "/* _______________ DEFINITIONS __________________ */\nFIELD ADDRS = [A15..12] ; /* Z80 CPU Address lines */\n\n/* _______________ EQUATIONS ___________________ */\n/* Memory Addressing */\nROM = MREQ & ADDRS:[0000..1FFF] ; /* 8K ROM Addressing */\nVRAM = MREQ & ADDRS:[2000..2FFF] ; /* 4K Video RAM Addressing */\nRAM = MREQ & ADDRS:[3000..3FFF] ; /* 4K RAM Addressing */\n\n/* I/O Addressing */\nIO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"
- moved on the sheet: C1, C11, C12, C2, C3, C5, C6, C7, C8, C9, D1, D2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

Commit message: Video improvement (#6)
* Preparing for expansion

* PLD update for expansion

* PLD update
Parts:
- removed H4: MountingHole, Mounting_Holes:MountingHole_3.2mm_M3, symbol Mechanical:MountingHole
- removed J3: TAPE, Sockets_MOLEX_KK-System:Socket_MOLEX-KK-RM2-54mm_Lock_3pin_straight, symbol Connector:Conn_01x03_Male
- removed U2: 27C64, Housings_DIP:DIP-28_W15.24mm_Socket, symbol Memory_EPROM:2764
- added J3: Conn_01x03, Pin_Headers:Pin_Header_Angled_1x03_Pitch2.54mm, symbol Connector_Generic:Conn_01x03
- added JP2: Jumper, Connector_PinHeader_2.54mm:PinHeader_1x02_P2.54mm_Vertical, symbol Device:Jumper
- added R58: 10k, Resistor_SMD:R_0805_2012Metric_Pad1.15x1.40mm_HandSolder, symbol Device:R
- added U2: 27C128, Package_DIP:DIP-28_W15.24mm, symbol Memory_EPROM:27C128
- C12: value 22u -> 10u
- C7, C8, C9: footprint Capacitors_SMD:C_0805_HandSoldering -> Capacitor_SMD:C_0805_2012Metric_Pad1.15x1.40mm_HandSolder
- J5: footprint Connectors:BARREL_JACK -> Connector_BarrelJack:BarrelJack_Horizontal
- R1, R10, R11, R12, R13, R14, R2, R3, R4, R5, R56, R6, R7, R8, R9: footprint Resistors_SMD:R_0805_HandSoldering -> Resistor_SMD:R_0805_2012Metric_Pad1.15x1.40mm_HandSolder
Connections:
- net +5V: now also R58.1, U2.1 (VPP), U2.27 (~PGM), U2.28 (VCC)
- net A0: now also U2.10 (A0)
- net A1: now also U2.9 (A1)
- net A10: now also U2.21 (A10)
- net A11: now also U2.23 (A11)
- net A12: now also U2.2 (A12)
- net A2: now also U2.8 (A2)
- net A3: now also U2.7 (A3)
- net A4: now also U2.6 (A4)
- net A5: now also U2.5 (A5)
- net A6: now also U2.4 (A6)
- net A7: now also U2.3 (A7)
- net A8: now also U2.25 (A8)
- net A9: now also U2.24 (A9)
- net D0: now also U2.11 (D0)
- net D1: now also U2.12 (D1)
- net D2: now also U2.13 (D2)
- net D3: now also U2.15 (D3)
- net D4: now also U2.16 (D4)
- net D5: now also U2.17 (D5)
- net D6: now also U2.18 (D6)
- net D7: now also U2.19 (D7)
- net GNDD: now also J3.2 (Pin_2), JP2.1, U2.14 (GND)
- net ~RD: now also U2.22 (~OE)
- net ~ROMSL: now also U2.20 (~CE)
- net at C8.1, R13.1, R14.2: now also J3.3 (Pin_3)
- net at C7.1, R12.1: now also J3.1 (Pin_1)
- net SPEAKER: now reaches J1.48 (Pin_48)
- new net: JP2.2, R58.2, U2.26 (A13)
- no-connect marks 6 -> 5
Other:
- note added: "Code\nSelection"
- moved on the sheet: R5
