File: Video.sch (KiCad schematic (older format))
At the start: 65 parts, among them J4 A/V, J6 Conn_02x15_Odd_Even, Q1 BC817, Q2 BC817, U10 74LS367, U11 74LS367, U12 74LS367, U13 74LS367, U14 GAL22V10, U7 74LS166, U8 6116, U9 6116, Y1 6.55 MHz

Commit message: Inverted video option
Parts:
- added JP1: Jumper, Pin_Headers:Pin_Header_Straight_1x02_Pitch2.54mm, symbol Device:Jumper
- added R57: 10k, Resistors_SMD:R_0805_HandSoldering, symbol Device:R
Connections:
- net +5V: now also R57.2
- net BLANK: now also JP1.1
- net ~WBKGND: now reaches U14.13 (I)
- net ~WBKGND: now also JP1.2, R57.1
- no-connect marks 8 -> 7
Other:
- note added: "Black on White\nVideo"
- note removed: "/* _______________ EQUATIONS _____________________ */\nVCLK = !OSC ; /* Video Clock */\nCHRRAM = !(SCRADR & !A11) ; /* Char Set RAM Enable */\nSCRRAM = !(SCRADR & CHRRAM) ; /* Screen RAM Enable */\nCHRADR = !SCRRAM ; /* Char Set RAM CPU Addressing */\nVRAMWR = SCRADR & WR ; /* Char and Screen RAM Write Enable */\nVLOAD = VIDEN & RGTPIX ; /* Load Video Shift Register */\nVHOLD = VIDEN & A10 ; /* V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"
- moved on the sheet: C10, C13, C14, C15, C16, C17, C20, C22, C23, D10, D9, J4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

Commit message: Video improvement (#6)
* Preparing for expansion

* PLD update for expansion

* PLD update
Parts:
- removed J4: A/V, Sockets_MOLEX_KK-System:Socket_MOLEX-KK-RM2-54mm_Lock_3pin_straight, symbol Connector:Conn_01x03_Male
- added J4: Conn_01x03, Connectors_Molex:Molex_KK-6410-03_03x2.54mm_Straight, symbol Connector_Generic:Conn_01x03
- C22, C23: footprint Capacitors_SMD:C_0805_HandSoldering -> Capacitor_SMD:C_0805_2012Metric_Pad1.15x1.40mm_HandSolder
- R15, R16, R17, R18, R19, R20, R21, R22, R23, R24, R25, R26, R27, R28, R29, R30, R31, R32, R33, R34, R35, R36, R37, R38, R39, R40, R41, R42, R43, R44, R45, R46, R47, R48, R49, R51, R52, R53, R54, R55, R57: footprint Resistors_SMD:R_0805_HandSoldering -> Resistor_SMD:R_0805_2012Metric_Pad1.15x1.40mm_HandSolder
- R50: value 4k7 -> 1k5; footprint Resistors_SMD:R_0805_HandSoldering -> Resistor_SMD:R_0805_2012Metric_Pad1.15x1.40mm_HandSolder
Connections:
- net OSC is gone; now on net VCLK: C22.1, Q1.3 (C), R50.2, R51.1, U14.11 (I)
- net GNDD: now also J4.2 (Pin_2)
- net INV: now also U14.14 (I/O); no longer U14.22 (I/O)
- net VCLK: no longer U14.14 (I/O)
- net VIDEN: no longer J6.27 (Pin_27)
- net SPEAKER: now reaches C10.2
- net SPEAKER: now also J4.1 (Pin_1)
- net at R55.1: now also J4.3 (Pin_3)
- new net BORDER: J6.27 (Pin_27), U14.22 (I/O)
