File: Jupiter-II_keyboard/Jupiter-II_keyboard.kicad_pcb (KiCad board)
At the start: 2 copper layers, 157.5 x 70.5 mm, 47 parts, among them J1 Conn_02x08_Odd_Even, SW1 1, SW10 0, SW11 Q, SW12 W, SW13 E, SW14 R, SW15 T, SW16 Y, SW17 U, SW18 I, SW19 O, SW2 2, SW20 P, SW21 A, SW22 S, SW23 D, SW24 F, SW25 G, SW26 H, SW27 J, SW28 K, SW29 L, SW3 3, SW30 ENTER, SW31 SHIFT, SW32 SYMBOL, SW33 Z, SW34 X, SW35 C, SW36 V, SW37 B, SW38 N, SW39 M, SW4 4, SW40 SPACE, SW5 5, SW6 6, SW7 7, SW8 8, SW9 9

Commit message: Keyboard redimensioning (#7)
* Resizing Board

* production gerbers
Parts:
- D1: footprint LEDs:LED_1206_HandSoldering -> LED_SMD:LED_1206_3216Metric_Pad1.42x1.75mm_HandSolder
- J1: footprint Connectors_Multicomp:Multicomp_MC9A12-1634_2x08x2.54mm_Straight -> Connector_IDC:IDC-Header_2x08_P2.54mm_Vertical
- R1: footprint Resistors_SMD:R_0805_HandSoldering -> Resistor_SMD:R_0805_2012Metric_Pad1.15x1.40mm_HandSolder
- SW1, SW10, SW11, SW12, SW13, SW14, SW15, SW16, SW17, SW18, SW19, SW2, SW20, SW21, SW22, SW23, SW24, SW25, SW26, SW27, SW28, SW29, SW3, SW30, SW31, SW32, SW33, SW34, SW35, SW36, SW37, SW38, SW39, SW4, SW40, SW5, SW6, SW7, SW8, SW9: footprint Buttons_Switches_THT:SW_PUSH_6mm -> Button_Switch_THT:SW_PUSH_6mm
- moved H3 1.91 mm to (55.2, 108.6)
- moved H4 1.91 mm to (203.8, 108.6)
- moved D1 1.27 mm to (129.5, 48.9)
- moved R1 1.27 mm to (98.4, 48.9)
- moved H1 1.27 mm to (55.2, 50.2)
- moved H2 1.27 mm to (203.8, 50.2)
- moved J1 1.27 mm to (71.8, 52.7), turned to 90 degrees
Routing:
- net /KA8: track 185.8 -> 181.6 mm
- net /KD0: track 288.0 -> 284.6 mm
- net /KD3: track 291.5 -> 288.8 mm
- net /KD4: track 217.5 -> 214.9 mm
- net /KD2: track 243.2 -> 240.8 mm
- net /KD1: track 249.6 -> 247.3 mm
- net /KA15: track 221.6 -> 219.6 mm
- net /KA14: track 178.7 -> 176.7 mm
- net /KA13: track 139.1 -> 137.1 mm
- net /KA9: track 103.5 -> 102.2 mm
- net /KA10: track 89.5 -> 88.3 mm
- net /KA11: track 74.6 -> 73.5 mm
- net /KA12: track 116.3 -> 115.4 mm
- net Net-(D1-Pad2): track 27.8 -> 28.6 mm
Other:
- board size 157.5 x 70.5 mm -> 157.5 x 67.3 mm
- board text added: "June 2020 - Ricardo F. Lopes"
- board text removed: "2020 Ricardo F. Lopes"
