File: Jupiter-II_keyboard/Jupiter-II_keyboard.sch (KiCad schematic (older format))
At the start: 47 parts, among them J1 Conn_02x08_Odd_Even, SW1 1, SW10 0, SW11 Q, SW12 W, SW13 E, SW14 R, SW15 T, SW16 Y, SW17 U, SW18 I, SW19 O, SW2 2, SW20 P, SW21 A, SW22 S, SW23 D, SW24 F, SW25 G, SW26 H, SW27 J, SW28 K, SW29 L, SW3 3, SW30 ENTER, SW31 SHIFT, SW32 SYMBOL, SW33 Z, SW34 X, SW35 C, SW36 V, SW37 B, SW38 N, SW39 M, SW4 4, SW40 SPACE, SW5 5, SW6 6, SW7 7, SW8 8, SW9 9

Commit message: Keyboard redimensioning (#7)
* Resizing Board

* production gerbers
Parts:
- D1: footprint LEDs:LED_1206_HandSoldering -> LED_SMD:LED_1206_3216Metric_Pad1.42x1.75mm_HandSolder
- J1: footprint Connectors_Multicomp:Multicomp_MC9A12-1634_2x08x2.54mm_Straight -> Connector_IDC:IDC-Header_2x08_P2.54mm_Vertical
- R1: footprint Resistors_SMD:R_0805_HandSoldering -> Resistor_SMD:R_0805_2012Metric_Pad1.15x1.40mm_HandSolder
- SW1, SW10, SW11, SW12, SW13, SW14, SW15, SW16, SW17, SW18, SW19, SW2, SW20, SW21, SW22, SW23, SW24, SW25, SW26, SW27, SW28, SW29, SW3, SW30, SW31, SW32, SW33, SW34, SW35, SW36, SW37, SW38, SW39, SW4, SW40, SW5, SW6, SW7, SW8, SW9: footprint Buttons_Switches_THT:SW_PUSH_6mm -> Button_Switch_THT:SW_PUSH_6mm
